Commit message: Lots of updates

File: robot.xacro (robot description, xacro)
@@ -17,5 +17,5 @@
 	<xacro:property name="suspension_damping" value="1000.0" />
 	<xacro:property name="suspension_stiffness" value="100.0" />
-	<xacro:property name="max_steering_angle" value="0.5" />
+	<xacro:property name="max_steering_angle" value="1.5" />
 	<!-- Materials -->
 	<material name="blue">
@@ -30,6 +30,6 @@
 			<visual>
 				<geometry>
-					<!-- <mesh filename="./wheels/wheel_and_tire.dae" scale="2.0 2.0 2.0" /> -->
-					<cylinder radius="${wheel_radius}" length="${wheel_width}"/>
+					<mesh filename="./wheels/wheel_and_tire.dae" scale="2.0 2.0 2.0" />
+					<!-- <cylinder radius="${wheel_radius}" length="${wheel_width}"/> -->
 				</geometry>
 				<material name="black"/>

Commit message: updates

File: robot.xacro (robot description, xacro)
@@ -3,6 +3,6 @@
 	<xacro:arg name="suspend" default="true" />
 	<!-- Vehicle parameters -->
-	<xacro:property name="chassis_length" value="0.4" />
-	<xacro:property name="chassis_width" value="0.125" />
+	<xacro:property name="chassis_length" value="0.5" />
+	<xacro:property name="chassis_width" value="0.15" />
 	<xacro:property name="chassis_height" value="0.05" />
 	<xacro:property name="chassis_mass" value="8.0" />
@@ -11,7 +11,7 @@
 	<xacro:property name="wheel_mass" value="0.5" />
 	<!-- Distance between front and rear axles -->
-	<xacro:property name="wheelbase" value=".25" />
+	<xacro:property name="wheelbase" value="0.535" />
 	<!-- Distance between left and right wheels -->
-	<xacro:property name="track_width" value="0.25" />
+	<xacro:property name="track_width" value="0.281" />
 	<xacro:property name="suspension_travel" value="0.1" />
 	<xacro:property name="suspension_damping" value="1000.0" />
